File: hardware/coffee_esp32/coffee_esp32.kicad_sch (KiCad schematic)
At the start: 24 parts, among them Q2 TIP120, SW0 Power Switch, SW1 Power Switch, SW2 Power Switch, SW3 Power Switch, SW4 Power Switch, U1 ESP32-DEVKIT-V1

Commit message: load cell testing tares and calibrates
Connections:
- net Button 0: no longer U1.9 (D18)
- net Load Cell DOUT: now also U1.6 (RX2); no longer U1.19 (D34)
- net Load Cell SCK: now also U1.7 (TX2); no longer U1.20 (D35)
- net SPI MISO Bean: no longer INTAKE_AMP1.7 (DO), U1.15 (D23)
- net SPI SCK Intake renamed SPI SCK
- net SPI SCK: now also U1.9 (D18)
- new net SPI MISO: U1.15 (D23)
- new net SPI MISO Intake: INTAKE_AMP1.7 (DO)
- no-connect marks 20 -> 18
Changed lines of the file:
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@@
-	)
-	(junction
-		(at 189.23 105.41)
-		(diameter 0)
-		(color 0 0 0 0)
 	)
 	(junction
@@
 	)
 	(junction
-		(at 139.7 120.65)
-		(diameter 0)
-		(color 0 0 0 0)
-	)
-	(junction
 		(at 52.07 73.66)
 		(diameter 0)
@@
 	)
 	(no_connect
-		(at 180.34 95.25)
-	)
-	(no_connect
 		(at 87.63 139.7)
 	)
@@
 	)
 	(no_connect
-		(at 180.34 97.79)
-	)
-	(no_connect
 		(at 149.86 90.17)
 	)
@@
 	(wire
 		(pts
-			(xy 180.34 102.87) (xy 181.61 102.87)
-		)
-		(stroke
-			(width 0)
-			(type default)
-		)
-	)
-	(wire
-		(pts
 			(xy 83.82 74.93) (xy 85.09 74.93)
 		)
@@
 	(wire
 		(pts
-			(xy 189.23 105.41) (xy 191.77 105.41)
-		)
-		(stroke
-			(width 0)
-			(type default)
-		)
-	)
-	(wire
-		(pts
-			(xy 180.34 105.41) (xy 189.23 105.41)
-		)
-		(stroke
-			(width 0)
-			(type default)
-		)
-	)
-	(wire
-		(pts
 			(xy 180.34 80.01) (xy 182.88 80.01)
 		)
@@
 	(wire
 		(pts
-			(xy 189.23 102.87) (xy 191.77 102.87)
-		)
-		(stroke
-			(width 0)
-			(type default)
-		)
-	)
-	(wire
-		(pts
 			(xy 83.82 83.82) (xy 83.82 82.55)
 		)
@@
 	(wire
 		(pts
-			(xy 138.43 118.11) (xy 139.7 118.11)
-		)
-		(stroke
-			(width 0)
-			(type default)
-		)
-	)
-	(wire
-		(pts
 			(xy 223.52 91.44) (xy 223.52 92.71)
 		)
@@
 	(wire
 		(pts
-			(xy 189.23 105.41) (xy 189.23 102.87)
-		)
-		(stroke
-			(width 0)
-			(type default)
-		)
-	)
-	(wire
-		(pts
 			(xy 83.82 87.63) (xy 85.09 87.63)
 		)
@@
 	(wire
 		(pts
-			(xy 180.34 120.65) (xy 181.61 120.65)
-		)
-		(stroke
-			(width 0)
-			(type default)
-		)
-	)
-	(wire
-		(pts
 			(xy 260.35 81.28) (xy 260.35 82.55)
 		)
@@
 	(wire
 		(pts
-			(xy 180.34 123.19) (xy 181.61 123.19)
-		)
-		(stroke
-			(width 0)
-			(type default)
-		)
-	)
-	(wire
-		(pts
 			(xy 180.34 34.29) (xy 181.61 34.29)
 		)
@@
 	(wire
 		(pts
-			(xy 139.7 120.65) (xy 149.86 120.65)
-		)
-		(stroke
-			(width 0)
-			(type default)
-		)
-	)
-	(wire
-		(pts
 			(xy 33.02 34.29) (xy 41.91 34.29)
 		)
@@
 	(wire
 		(pts
-			(xy 139.7 120.65) (xy 139.7 118.11)
-		)
-		(stroke
-			(width 0)
-			(type default)
-		)
-	)
-	(wire
-		(pts
 			(xy 83.82 43.18) (xy 83.82 44.45)
-		)
-		(stroke
-			(width 0)
-			(type default)
-		)
-	)
-	(wire
-		(pts
-			(xy 138.43 120.65) (xy 139.7 120.65)
 		)
 		(stroke
@@
 		)
 	)
-	(label "SPI SCK Bean"
-		(at 124.46 120.65 0)
-		(effects
-			(font
-				(size 1.27 1.27)
-			)
-			(justify left bottom)
-		)
-	)
-	(label "SPI SCK Intake"
-		(at 124.46 118.11 0)
+	(label "I2C SCL"
+		(at 180.34 102.87 0)
 		(effects
 			(font
@@
 		)
 	)
+	(label "SPI MISO"
+		(at 180.34 105.41 0)
+		(effects
+			(font
+				(size 1.27 1.27)
+			)
+			(justify left bottom)
+		)
+	)
 	(label "Fan Base"
 		(at 181.61 107.95 0)
@@
 		)
 	)
-	(label "SPI MISO Intake"
-		(at 191.77 105.41 0)
-		(effects
-			(font
-				(size 1.27 1.27)
-			)
-			(justify left bottom)
-		)
-	)
 	(label "SPI CS Intake"
 		(at 134.62 105.41 0)
@@
 		)
 	)
-	(label "Load Cell DOUT"
-		(at 181.61 123.19 0)
-		(effects
-			(font
-				(size 1.27 1.27)
-			)
-			(justify left bottom)
-		)
-	)
 	(label "SPI SCK Bean"
 		(at 113.03 49.53 0)
@@
 		)
 	)
-	(label "I2C SCL"
-		(at 181.61 102.87 0)
-		(effects
-			(font
-				(size 1.27 1.27)
-			)
-			(justify left bottom)
-		)
-	)
 	(label "SPI SCK"
 		(at 149.86 120.65 180)
@@
 		)
 	)
+	(label "Load Cell DOUT"
+		(at 180.34 95.25 0)
+		(effects
+			(font
+				(size 1.27 1.27)
+			)
+			(justify left bottom)
+		)
+	)
 	(label "I2C SDA"
 		(at 149.86 49.53 180)
@@
 	)
 	(label "Load Cell SCK"
-		(at 181.61 120.65 0)
+		(at 180.34 97.79 0)
 		(effects
 			(font
@@
 		)
 	)
-	(label "SPI SCK Intake"
+	(label "SPI SCK"
 		(at 114.3 85.09 0)
 		(effects
@@
 		(effects
 			(font
-				(size 1.27 1.27)
-			)
-			(justify left bottom)
-		)
-	)
-	(label "SPI MISO Bean"
-		(at 191.77 102.87 0)
-		(effects
-			(font
